File: stathat.kicad_pcb (KiCad board)
At the start: 4 copper layers, 65 x 56.5 mm, 44 parts, among them J1 Conn_01x01, J2 Conn_01x01, J3 Conn_01x01, J4 Raspberry_Pi_2_3, J5 Conn_01x01, J6 Conn_01x01, J7 Conn_01x01, J8 Conn_01x01, J9 Conn_01x01, U1 LTV-844S, U2 74HC14

Commit message: minor DRC and ERC cleanup. updated render
Other:
- board text added: "FOSS || GTFO"
Changed lines of the file:
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@@
 			(plotpadnumbers no)
 			(hidednponfab no)
-			(sketchdnponfab yes)
-			(crossoutdnponfab yes)
+			(sketchdnponfab no)
+			(crossoutdnponfab no)
 			(subtractmaskfromsilk yes)
 			(outputformat 1)
@@
 			)
 		)
-		(property "DK" ""
+		(property "DK" "311-2.20KLRCT-ND"
 			(at 0 0 270)
 			(unlocked yes)
@@
 			)
 		)
-		(property "PARTNO" ""
+		(property "PARTNO" "RC0402FR-072K2L"
 			(at 0 0 270)
 			(unlocked yes)
@@
 			)
 		)
-		(property "DK" ""
+		(property "DK" "1276-1040-1-ND"
 			(at 0 0 0)
 			(unlocked yes)
@@
 			)
 		)
-		(property "PARTNO" ""
+		(property "PARTNO" "CL10A225KO8NNNC"
 			(at 0 0 0)
 			(unlocked yes)
@@
 			)
 		)
-		(property "Description" ""
+		(property "Description" "Mounting Hole without connection"
 			(at 0 0 270)
 			(unlocked yes)
@@
 			)
 		)
-		(property "DK" ""
+		(property "DK" "311-2.20KLRCT-ND"
 			(at 0 0 270)
 			(unlocked yes)
@@
 			)
 		)
-		(property "PARTNO" ""
+		(property "PARTNO" "RC0402FR-072K2L"
 			(at 0 0 270)
 			(unlocked yes)
@@
 			)
 		)
-		(property "DK" ""
+		(property "DK" "1276-1040-1-ND"
 			(at 0 0 0)
 			(unlocked yes)
@@
 			)
 		)
-		(property "PARTNO" ""
+		(property "PARTNO" "CL10A225KO8NNNC"
 			(at 0 0 0)
 			(unlocked yes)
@@
 			)
 		)
-		(property "DK" ""
+		(property "DK" "1276-1040-1-ND"
 			(at 0 0 0)
 			(unlocked yes)
@@
 			)
 		)
-		(property "PARTNO" ""
+		(property "PARTNO" "CL10A225KO8NNNC"
 			(at 0 0 0)
 			(unlocked yes)
@@
 			)
 		)
-		(property "Description" ""
+		(property "Description" "Light emitting diode, filled shape"
 			(at 0 0 90)
 			(layer "F.Fab")
@@
 			)
 		)
+		(property "Sim.Pins" "1=K 2=A"
+			(at 0 0 90)
+			(unlocked yes)
+			(layer "F.Fab")
+			(hide yes)
+			(effects
+				(font
+					(size 1 1)
+					(thickness 0.15)
+				)
+			)
+		)
 		(property ki_fp_filters "LED* LED_SMD:* LED_THT:*")
 		(sheetname "/")
@@
 			)
 		)
-		(property "DK" ""
+		(property "DK" "13-RC1210FR-075K1LCT-ND"
 			(at 0 0 270)
 			(unlocked yes)
@@
 			)
 		)
-		(property "PARTNO" ""
+		(property "PARTNO" "RC1210FR-075K1L"
 			(at 0 0 270)
 			(unlocked yes)
@@
 			)
 		)
-		(property "DK" ""
+		(property "DK" "13-RC1210FR-075K1LCT-ND"
 			(at 0 0 270)
 			(unlocked yes)
@@
 			)
 		)
-		(property "PARTNO" ""
+		(property "PARTNO" "RC1210FR-075K1L"
 			(at 0 0 270)
 			(unlocked yes)
@@
 			)
 		)
-		(property "Description" ""
+		(property "Description" "Mounting Hole without connection"
 			(at 0 0 270)
 			(unlocked yes)
@@
 			)
 		)
+		(property "PARTNO" "SN74HC14DR"
+			(at 0 0 180)
+			(unlocked yes)
+			(layer "F.Fab")
+			(hide yes)
+			(effects
+				(font
+					(size 1 1)
+					(thickness 0.15)
+				)
+			)
+		)
+		(property "DK" "296-1194-1-ND"
+			(at 0 0 180)
+			(unlocked yes)
+			(layer "F.Fab")
+			(hide yes)
+			(effects
+				(font
+					(size 1 1)
+					(thickness 0.15)
+				)
+			)
+		)
 		(property ki_fp_filters "DIP*W7.62mm*")
 		(sheetname "/")
@@
 			(net "unconnected-(J4-GPIO27-Pad13)")
 			(pinfunction "GPIO27_13")
-			(pintype "bidirectional")
+			(pintype "bidirectional+no_connect")
 		)
 		(pad "14" thru_hole oval
@@
 			)
 		)
-		(property "DK" ""
+		(property "DK" "13-RC1210FR-075K1LCT-ND"
 			(at 0 0 270)
 			(unlocked yes)
@@
 			)
 		)
-		(property "PARTNO" ""
+		(property "PARTNO" "RC1210FR-075K1L"
 			(at 0 0 270)
 			(unlocked yes)
@@
 			)
 		)
-		(property "DK" ""
+		(property "DK" "13-RC1210FR-075K1LCT-ND"
 			(at 0 0 270)
 			(unlocked yes)
@@
 			)
 		)
-		(property "PARTNO" ""
+		(property "PARTNO" "RC1210FR-075K1L"
 			(at 0 0 270)
 			(unlocked yes)
@@
 			)
 		)
-		(property "Description" ""
+		(property "Description" "Light emitting diode, filled shape"
 			(at 0 0 90)
 			(layer "F.Fab")
@@
 			)
 		)
+		(property "Sim.Pins" "1=K 2=A"
+			(at 0 0 90)
+			(unlocked yes)
+			(layer "F.Fab")
+			(hide yes)
+			(effects
+				(font
+					(size 1 1)
+					(thickness 0.15)
+				)
+			)
+		)
 		(property ki_fp_filters "LED* LED_SMD:* LED_THT:*")
 		(sheetname "/")
@@
 			)
 		)
-		(property "DK" ""
+		(property "DK" "1276-1002-1-ND"
 			(at 0 0 0)
 			(unlocked yes)
@@
 			)
 		)
-		(property "PARTNO" ""
+		(property "PARTNO" "CL05B104KP5NNNC"
 			(at 0 0 0)
 			(unlocked yes)
@@
 			)
 		)
-		(property "Description" ""
+		(property "Description" "Light emitting diode, filled shape"
 			(at 0 0 90)
 			(layer "F.Fab")
@@
 			)
 		)
+		(property "Sim.Pins" "1=K 2=A"
+			(at 0 0 90)
+			(unlocked yes)
+			(layer "F.Fab")
+			(hide yes)
+			(effects
+				(font
+					(size 1 1)
+					(thickness 0.15)
+				)
+			)
+		)
 		(property ki_fp_filters "LED* LED_SMD:* LED_THT:*")
 		(sheetname "/")
@@
 			)
 		)
-		(property "DK" ""
+		(property "DK" "13-RC1210FR-075K1LCT-ND"
 			(at 0 0 90)
 			(unlocked yes)
@@
 			)
 		)
-		(property "PARTNO" ""
+		(property "PARTNO" "RC1210FR-075K1L"
 			(at 0 0 90)
 			(unlocked yes)
@@
 			)
 		)
-		(property "DK" ""
+		(property "DK" "1276-1040-1-ND"
 			(at 0 0 0)
 			(unlocked yes)
@@
 			)
 		)
-		(property "PARTNO" ""
+		(property "PARTNO" "CL10A225KO8NNNC"
 			(at 0 0 0)
 			(unlocked yes)
@@
 			)
 		)
-		(property "DK" ""
+		(property "DK" "311-2.20KLRCT-ND"
 			(at 0 0 270)
 			(unlocked yes)
@@
 			)
 		)
-		(property "PARTNO" ""
+		(property "PARTNO" "RC0402FR-072K2L"
 			(at 0 0 270)
 			(unlocked yes)
@@
 			)
 		)
-		(property "DK" ""
+		(property "DK" "13-RC1210FR-075K1LCT-ND"
 			(at 0 0 270)
 			(unlocked yes)
@@
 			)
 		)
-		(property "PARTNO" ""
+		(property "PARTNO" "RC1210FR-075K1L"
 			(at 0 0 270)
 			(unlocked yes)
@@
 			)
 		)
-		(property "DK" ""
+		(property "DK" "13-RC1210FR-075K1LCT-ND"
 			(at 0 0 270)
 			(unlocked yes)
@@
 			)
 		)
-		(property "PARTNO" ""
+		(property "PARTNO" "RC1210FR-075K1L"
 			(at 0 0 270)
 			(unlocked yes)
@@
 			)
 		)
-		(property "Description" ""
+		(property "Description" "Mounting Hole without connection"
 			(at 0 0 270)
 			(unlocked yes)
@@
 			)
 		)
-		(property "DK" ""
+		(property "DK" "13-RC1210FR-075K1LCT-ND"
 			(at 0 0 270)
 			(unlocked yes)
@@
 			)
 		)
-		(property "PARTNO" ""
+		(property "PARTNO" "RC1210FR-075K1L"
 			(at 0 0 270)
 			(unlocked yes)
@@
 			)
 		)
-		(property "DK" ""
+		(property "DK" "311-2.20KLRCT-ND"
 			(at 0 0 270)
 			(unlocked yes)
@@
 			)
 		)
-		(property "PARTNO" ""
+		(property "PARTNO" "RC0402FR-072K2L"
 			(at 0 0 270)
 			(unlocked yes)
@@
 			)
 		)
-		(property "Description" ""
+		(property "Description" "Mounting Hole without connection"
 			(at 0 0 270)
 			(unlocked yes)
@@
 			)
 		)
-		(property "Description" ""
+		(property "Description" "Light emitting diode, filled shape"
 			(at 0 0 90)
 			(layer "F.Fab")
@@
 			)
 		)
+		(property "Sim.Pins" "1=K 2=A"
+			(at 0 0 90)
+			(unlocked yes)
+			(layer "F.Fab")
+			(hide yes)
+			(effects
+				(font
+					(size 1 1)
+					(thickness 0.15)
+				)
+			)
+		)
 		(property ki_fp_filters "LED* LED_SMD:* LED_THT:*")
 		(sheetname "/")
@@
 		(layer "Edge.Cuts")
 	)
+	(gr_text "FOSS || GTFO"
+		(at 154.65 118.425 0)
+		(layer "F.Cu")
+		(effects
+			(font
+				(size 1 1)
+				(thickness 0.15)
+			)
+			(justify left bottom)
+		)
+	)
 	(gr_text "R"

Commit message: add fix for #1. move all vias out of pads. clean up traces. bump version number
Parts:
- removed U1: LTV-844S, Package_SO:SOIC-16W_7.5x10.3mm_P1.27mm
- added TP13: GND, stathat:TestPoint_Pad_D1.0mm, F.Cu at (165.9, 108.0)
- added U4: LTV-844S, stathat:OPTO-SMD-16_L19.8-W6.5-P2.54-LS10.2-BL, F.Cu at (153.7, 100.2)
- moved TP12 8.66 mm to (165.9, 95.6)
- moved TP9 8.66 mm to (165.9, 98.7)
- moved TP11 8.66 mm to (165.9, 101.8)
- moved TP10 8.66 mm to (165.9, 104.9)
- moved C2 8.23 mm to (157.6, 109.6)
- moved R10 8.23 mm to (154.1, 108.3)
- moved R2 8.23 mm to (159.2, 108.3)
- moved C1 8.23 mm to (160.1, 109.6)
- moved C3 8.23 mm to (155.1, 109.6)
- moved R6 8.23 mm to (156.6, 108.3)
Routing:
- net /THERM_FAN_RAW: track 30.1 -> 43.6 mm
- net Net-(U4-AC1): track 19.3 -> 8.14 mm
- net /THERM_HEAT2_RAW: track 37.8 -> 48.4 mm
- net /THERM_HEAT_RAW: track 30.7 -> 39.8 mm
- net /THERM_COOL_RAW: track 29.5 -> 37.3 mm
- net Net-(U4-CA1): track 14.7 -> 8.54 mm
- net /GND: track 10.9 -> 16.8 mm, vias 14 -> 15
- net Net-(U4-AC3): track 10.1 -> 15.2 mm
- net /-24VAC: track 57.8 -> 62.8 mm
- net Net-(U4-CA3): track 14.5 -> 18.4 mm
- net Net-(U4-CA2): track 8.48 -> 11.6 mm
- net Net-(U4-AC4): track 18.4 -> 21.4 mm
- net Net-(U4-CA4): track 21.7 -> 22.9 mm
- net /THERM_COOL: track 31.5 -> 32.6 mm
- net /THERM_HEAT2: track 26.1 -> 26.6 mm
Other:
- board text added: "StatHat v2"
- board text removed: "StatHat v1"
